File: circuit/schematic.kicad_pcb (KiCad board)
At the start: 2 copper layers, 104.2 x 54.2 mm, 62 parts, among them IC1 SN74LVC2G14DBVR, J1 DIN-5, J2 DIN-5, J3 Barrel_Jack_Switch, J4 DIN-6, J5 AudioJack3_Dual_Switch, SW1 SW_Push, SW2 SW_Push, U1 ATtiny841-SSU, U2 6N138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

Commit message: Add board rev.2
Parts:
- added J6: AudioJack3_Dual_Switch, NYS_Jacks:NYS2152, F.Cu at (220.4, 7.72)
- added K1: V23079A1001B301, V23079A1001B301:V23079A1001B301, F.Cu at (292.1, 53.1)
- added K2: V23079A1001B301, V23079A1001B301:V23079A1001B301, F.Cu at (292.1, 63.4)
- C3: footprint Capacitor_SMD:C_0603_1608Metric_Pad1.05x0.95mm_HandSolder -> Capacitor_SMD:C_0603_1608Metric_Pad1.08x0.95mm_HandSolder
Connections:
- J1 pad MH: Net-(C2-Pad1) -> (no net)
- J2 pad MH: GND -> (no net)
